Commit message: Update ROS control and description for Unity integration

File: src/robotic_description/urdf/adaptive_gripper_arm.urdf (robot description, URDF)
Before this commit: robot adaptive_gripper_arm, 10 links, 9 joints
Joints:
- joint elbow_joint: limit lower=-1.5708 upper=1.5708 effort=4.0 velocity=1.5 -> lower=0.0 upper=1.5708 effort=4.0 velocity=1.2
- joint finger_left_joint: limit lower=0.0 upper=1.5708 effort=2.0 velocity=2.0 -> lower=0.0 upper=1.2217 effort=2.0 velocity=1.5
- joint finger_right_joint: mimic joint=finger_left_joint multiplier=1.0 offset=0.0 -> (none)
- joint shoulder_joint: limit lower=-1.5708 upper=1.5708 effort=5.0 velocity=1.5 -> lower=-1.0472 upper=1.0472 effort=5.0 velocity=1.2
- joint wrist_joint: axis 0 1 0 -> 0 0 1; limit lower=-1.5708 upper=1.5708 effort=3.0 velocity=2.0 -> lower=-1.0472 upper=1.0472 effort=3.0 velocity=1.5
